Commit message: feat:换掉了旧的urdf模型,,不过训了七百轮还没收敛

File: source/IRobot_wl/data/Robots/wl/wl_description/urdf/wl.urdf (robot description, URDF)
Before this commit: robot wl, 7 links, 6 joints
Links:
- link base_link: mass 8.8 -> 9.92239814270616
- link l_wheel_Link: mass 1.22 -> 0.177580655363663; geometry collision mesh filename=../meshes/l_wheel_Link.STL; visual mesh filename=../meshes/l_wheel_Link.STL
- link lf0_Link: mass 0.16 -> 0.22671
- link lf1_Link: mass 0.36 -> 0.22939
- link r_wheel_Link: mass 1.22 -> 0.177580658617343; geometry collision mesh filename=../meshes/r_wheel_Link.STL; visual mesh filename=../meshes/r_wheel_Link.STL
- link rf0_Link: mass 0.16 -> 0.237147723000171
- link rf1_Link: mass 0.36 -> 0.229390429090394
Joints:
- joint l_wheel_Joint: limit effort=5 velocity=1000 -> (none); origin xyz=1.857E-05 0.25 0.0275 rpy=0 0 0 -> xyz=-0.210696556901918 0.141859628740362 -0.00599999999999937 rpy=0 0 0; type revolute -> continuous
- joint lf0_Joint: limit lower=-0.3363 upper=1.3479 effort=30 velocity=1000 -> (none); origin xyz=0.054 0.1705 0.131 rpy=-1.5708 0 0 -> xyz=-0.0077481 0.16652 0.014601 rpy=-1.5708 0 0; type revolute -> continuous
- joint lf1_Joint: limit lower=-1.0 upper=1.25 effort=30 velocity=1000 -> lower=-0.6 upper=0.2 effort=40 velocity=1000; origin xyz=0.15 -0.00010199 0.0205 rpy=0 0 0 -> xyz=0.21472 0.029422 0.0062402 rpy=0 0 0
- joint r_wheel_Joint: limit effort=5 velocity=1000 -> (none); origin xyz=1.5909E-05 -0.25 0.0275 rpy=0 0 0 -> xyz=-0.210696556901869 -0.141859628740493 -0.00599999999999556 rpy=0 0 0; type revolute -> continuous
- joint rf0_Joint: limit lower=-1.3479 upper=0.3363 effort=30 velocity=1000 -> (none); origin xyz=0.054 -0.1705 0.131 rpy=1.5708 0 0 -> xyz=-0.00767633558745229 -0.176803872353463 0.0142033835799731 rpy=1.5707963267949 0 0; type revolute -> continuous
- joint rf1_Joint: limit lower=-1.25 upper=1.0 effort=30 velocity=1000 -> lower=-0.2 upper=0.6 effort=40 velocity=1000; origin xyz=0.15 9.5536E-05 0.0205 rpy=0 0 0 -> xyz=0.21416 -0.032328 0.0062402 rpy=0 0 0

Commit message: fix:继续修方向问题,修了轮子方向

File: source/IRobot_wl/data/Robots/wl/wl_description/urdf/wl.urdf (robot description, URDF)
Before this commit: robot wl, 7 links, 6 joints
Links:
- link l_wheel_Link: geometry collision cylinder length=0.0487 radius=0.058; visual mesh filename=../meshes/l_wheel_Link.STL
- link r_wheel_Link: geometry collision cylinder length=0.0487 radius=0.058; visual mesh filename=../meshes/r_wheel_Link.STL
